File: STUSB4500-EvalBoard/PCB/STUSB4500.brd (EAGLE design)
At the start: 16 x 24 mm, 25 parts

Commit message: Updated stusb part
Changed lines of the file:
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@@
 <drawing>
 <settings>
-<setting alwaysvectorfont="yes"/>
+<setting alwaysvectorfont="no"/>
 <setting verticaltext="up"/>
 </settings>
@@
 <contactref element="U$1" pad="22"/>
 <contactref element="U$1" pad="3"/>
-<wire x1="6.155625" y1="11.05" x2="6.223125" y2="10.9825" width="0.1524" layer="1"/>
 <wire x1="8.758125" y1="11.55" x2="7.23229375" y2="11.55" width="0.1524" layer="1"/>
 <wire x1="7.232290625" y1="11.55" x2="7.108125" y2="11.55" width="0.1524" layer="1"/>
@@
 <wire x1="11.05" y1="17.9" x2="11.35" y2="17.9" width="0.3048" layer="1"/>
 <wire x1="4.65" y1="17.9" x2="4.95" y2="17.9" width="0.3048" layer="1"/>
-<wire x1="6.608125" y1="11.05" x2="6.858125" y2="11.3" width="0.1524" layer="1"/>
 <via x="6.858125" y="11.3" extent="1-16" drill="0.3"/>
 <contactref element="R2" pad="1"/>
@@
 <wire x1="5.608125" y1="10.05" x2="5.746175" y2="10.18805" width="0.1524" layer="1"/>
 <wire x1="5.746175" y1="10.18805" x2="6.064375" y2="10.50625" width="0.1524" layer="1"/>
-<wire x1="4.958125" y1="11.05" x2="6.155625" y2="11.05" width="0.1524" layer="1"/>
 <via x="3.5" y="14" extent="1-16" drill="0.3"/>
 <contactref element="J5" pad="3"/>
@@
 <via x="10.8" y="1" extent="1-16" drill="0.3"/>
 <via x="5.1" y="1" extent="1-16" drill="0.3"/>
-<wire x1="6.608125" y1="11.05" x2="6.223125" y2="10.9825" width="0" layer="19" extent="1-1"/>
+<wire x1="6.858125" y1="11.3" x2="6.608125" y2="11.05" width="0.1524" layer="1"/>
+<wire x1="6.608125" y1="11.05" x2="4.958125" y2="11.05" width="0.1524" layer="1"/>
 </signal>
 <signal name="STUSB_RST">
@@
 <mfgpreviewcolor name="substratecolor" color="0xFF786E46"/>
 </mfgpreviewcolors>
+<errors>
+</errors>
 </board>
 </drawing>

Commit message: Cleanups in BOM, fixed OLED layout
Parts:
- C1, C2: value 1u -> 1uF 6.3V
- C3: value 100n -> 100n 25V
- C4: value 4.7u -> 10uF 25V
- C5: value 1u -> 10uF 25V
Changed lines of the file:
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@@
 </autorouter>
 <elements>
-<element name="C1" library="DD_rcl" package="C0402" package3d_urn="urn:adsk.eagle:package:23626/2" value="1u" x="10.668125" y="12.2525" smashed="yes">
+<element name="C1" library="DD_rcl" package="C0402" package3d_urn="urn:adsk.eagle:package:23626/2" value="1uF 6.3V" x="10.668125" y="12.2525" smashed="yes">
 <attribute name="POPULARITY" value="18" x="36.068125" y="-5.5275" size="1.778" layer="27" display="off"/>
 <attribute name="SPICEPREFIX" value="C" x="36.068125" y="-5.5275" size="1.778" layer="27" display="off"/>
 <attribute name="VALUE" x="9.398125" y="9.7125" size="1.27" layer="27"/>
 </element>
-<element name="C2" library="DD_rcl" package="C0402" package3d_urn="urn:adsk.eagle:package:23626/2" value="1u" x="10.668125" y="10.82375" smashed="yes">
+<element name="C2" library="DD_rcl" package="C0402" package3d_urn="urn:adsk.eagle:package:23626/2" value="1uF 6.3V" x="10.668125" y="10.82375" smashed="yes">
 <attribute name="POPULARITY" value="18" x="41.148125" y="-6.95625" size="1.778" layer="27" display="off"/>
 <attribute name="SPICEPREFIX" value="C" x="41.148125" y="-6.95625" size="1.778" layer="27" display="off"/>
 <attribute name="VALUE" x="9.398125" y="8.28375" size="1.27" layer="27"/>
 </element>
-<element name="C3" library="DD_rcl" package="C0402" package3d_urn="urn:adsk.eagle:package:23626/2" value="100n" x="9.6" y="5.2" smashed="yes">
+<element name="C3" library="DD_rcl" package="C0402" package3d_urn="urn:adsk.eagle:package:23626/2" value="100n 25V" x="9.6" y="5.2" smashed="yes">
 <attribute name="POPULARITY" value="18" x="29.92" y="-18.93" size="1.778" layer="27" display="off"/>
 <attribute name="SPICEPREFIX" value="C" x="29.92" y="-18.93" size="1.778" layer="27" display="off"/>
 <attribute name="VALUE" x="8.965" y="3.295" size="1.27" layer="27"/>
 </element>
-<element name="C4" library="DD_rcl" package="C1206" package3d_urn="urn:adsk.eagle:package:23618/2" value="4.7u" x="12.155625" y="15.4275" smashed="yes">
+<element name="C4" library="DD_rcl" package="C1206" package3d_urn="urn:adsk.eagle:package:23618/2" value="10uF 25V" x="12.155625" y="15.4275" smashed="yes">
 <attribute name="POPULARITY" value="54" x="40.095625" y="3.9975" size="1.778" layer="27" display="off"/>
 <attribute name="SPICEPREFIX" value="C" x="40.095625" y="3.9975" size="1.778" layer="27" display="off"/>
 <attribute name="VALUE" x="10.885625" y="12.8875" size="1.27" layer="27"/>
 </element>
-<element name="C5" library="DD_rcl" package="C1206" package3d_urn="urn:adsk.eagle:package:23618/2" value="1u" x="4.5" y="5.25" smashed="yes" rot="R90">
+<element name="C5" library="DD_rcl" package="C1206" package3d_urn="urn:adsk.eagle:package:23618/2" value="10uF 25V" x="4.5" y="5.25" smashed="yes" rot="R90">
 <attribute name="POPULARITY" value="54" x="15.93" y="38.27" size="1.778" layer="27" rot="R90" display="off"/>
 <attribute name="SPICEPREFIX" value="C" x="15.93" y="38.27" size="1.778" layer="27" rot="R90" display="off"/>
