File: STUSB4500-EvalBoard/PCB/STUSB4500.sch (EAGLE design)
At the start: 25 parts

Commit message: Cleanups in BOM, fixed OLED layout
Parts:
- C1, C2: value 1u -> 1uF 6.3V
- C3: value 100n -> 100n 25V
- C4: value 4.7u -> 10uF 25V
- C5: value 1u -> 10uF 25V
Other:
- moved on the sheet: C1, C2, R7
