File: STUSB4500-PowerSupply/PCB/STUSB4500_PS.brd (EAGLE design)
At the start: 60 x 40 mm, 101 parts, among them J2 FEMALE 2x3, J3 FEMALE 2x3, J4 FEMALE 2x3, SW1 SPST_TACT-EVQQ2

Commit message: Cleanups
Connections:
- net 3V3_IN renamed DC-DC-3V3
- net 3V3_OUT renamed DC-DC-3V3_OUT
- net 5V0_IN renamed DC-DC-5V0
- net 5V0_OUT renamed DC-DC-5V0_OUT
- net USB-PD_OUT renamed USB-PD_VDD_OUT
- net VDD renamed USB_PD_VDD*
Routing:
- net USB_PD_VDD: track 103.4 -> 106.4 mm
- net DC-DC-3V3: track 90.0 -> 90.7 mm
