File: STUSB4500-PowerSupply/PCB/STUSB4500_PS.brd (EAGLE design)
At the start: 60 x 40 mm, 101 parts, among them J2 FEMALE 2x3, J3 FEMALE 2x3, J4 FEMALE 2x3, SW1 SPST_TACT-EVQQ2

Commit message: Added reset pullup
Parts:
- added R1: 1k, DD_rcl:R0402
Connections:
- net +3V3: now also R1.2
- net NRST: now also R1.1
Routing:
- net GND: track 41.6 -> 26.3 mm, vias 184 -> 183
- net STUSB_AB: track 41.5 -> 41.6 mm, vias 3 -> 2
